File: Devboard.kicad_sch (KiCad schematic)
At the start: 40 parts, among them J1 USB_C_Receptacle_USB2.0_14P, J2 Conn_01x03, J3 Conn_01x10, J4 Conn_01x10, J5 JST_2mm_LiPo, J6 Conn_01x10, J7 Conn_01x10, SW1 SW_Push, U1 RP2040, U2 NCP1117-3.3_SOT223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

Commit message: Added an IMU, Solved all DRC thermal relief errors + routed IMU
Parts:
- added C19, C20, C21: 0.1uF, PCM_SparkFun-Capacitor:C_0603_1608Metric, symbol PCM_SparkFun-Capacitor:C
Connections:
- net GPIO21 is gone; now on net SDA: J7.7 (Pin_7), U1.32 (GPIO21)
- net GPIO22 is gone; now on net SCL: J7.9 (Pin_9), U1.34 (GPIO22)
- net +3.3V: now also U4.13 (VDD), U4.8 (VDDIO), C19.2, C20.1
- net GND: now also U4.18 (GND), U4.20 (RESV_GND), C19.1, C20.2, C21.2
- net at U4.10 (REGOUT): now also C21.1
- net SCL: now reaches U4.23 (SCL/SCLK)
- net SDA: now reaches U4.24 (SDA/MOSI)

Commit message: Changed IMU from MPU-6500 to ICM-20948
Parts:
- removed C21: 0.1uF, PCM_SparkFun-Capacitor:C_0603_1608Metric, symbol PCM_SparkFun-Capacitor:C
- removed U4: MPU-9250, Sensor_Motion:InvenSense_QFN-24_3x3mm_P0.4mm, symbol Sensor_Motion:MPU-9250
- added C22: 0.1uF, PCM_SparkFun-Capacitor:C_0603_1608Metric, symbol PCM_SparkFun-Capacitor:C
- added U4: ICM-20948, Sensor_Motion:InvenSense_QFN-24_3x3mm_P0.4mm, symbol Sensor_Motion:ICM-20948
Connections:
- net +3.3V: now also U4.13 (VDD); no longer C19.2
- net GND: now also C22.1, U4.18 (GND), U4.20 (GND)
- net SCL: now also U4.23 (SCL/SCLK)
- net SDA: now also U4.24 (SDA/SDI)
- new net: C22.2, U4.10 (REGOUT)
- new net 1.8V: C19.2, U4.8 (VDDIO)
Other:
- moved on the sheet: C19, C20

Commit message: Updated Devboard
Other:
- moved on the sheet: C19, C20, C22, U4

Commit message: Re-routed the board to a 2-layer PCB and removed IMU unit
Parts:
- removed C19, C20, C22: 0.1uF, PCM_SparkFun-Capacitor:C_0603_1608Metric, symbol PCM_SparkFun-Capacitor:C
- removed J3, J4, J6, J7: Conn_01x10, Connector_PinHeader_2.54mm:PinHeader_1x10_P2.54mm_Vertical, symbol Connector_Generic:Conn_01x10
- removed U4: ICM-20948, Sensor_Motion:InvenSense_QFN-24_3x3mm_P0.4mm, symbol Sensor_Motion:ICM-20948
- added J3, J4: Conn_01x20, Connector_PinHeader_2.54mm:PinHeader_1x20_P2.54mm_Vertical, symbol Connector_Generic:Conn_01x20
Connections:
- net +3.3V: now also J4.16 (Pin_16)
- net GND: now also J3.13 (Pin_13), J3.18 (Pin_18), J3.3 (Pin_3), J3.8 (Pin_8), J4.13 (Pin_13), J4.18 (Pin_18), J4.3 (Pin_3), J4.8 (Pin_8)
- net GPIO0: now also J3.1 (Pin_1)
- net GPIO1: now also J3.2 (Pin_2)
- net GPIO10: now also J3.14 (Pin_14)
- net GPIO11: now also J3.15 (Pin_15)
- net GPIO12: now also J3.16 (Pin_16)
- net GPIO13: now also J3.17 (Pin_17)
- net GPIO14: now also J3.19 (Pin_19)
- net GPIO15: now also J3.20 (Pin_20)
- net GPIO16: now also J4.1 (Pin_1)
- net GPIO17: now also J4.2 (Pin_2)
- net GPIO18: now also J4.4 (Pin_4)
- net GPIO19: now also J4.5 (Pin_5)
- net GPIO2: now also J3.4 (Pin_4)
- net GPIO20: now also J4.6 (Pin_6)
- net GPIO23: now also J4.11 (Pin_11)
- net GPIO24: now also J4.12 (Pin_12)
- net GPIO26_ADC0: now also J4.14 (Pin_14)
- net GPIO27_ADC1: now also J4.15 (Pin_15)
- net GPIO28_ADC2: now also J4.17 (Pin_17)
- net GPIO3: now also J3.5 (Pin_5)
- net GPIO4: now also J3.6 (Pin_6)
- net GPIO5: now also J3.7 (Pin_7)
- net GPIO6: now also J3.9 (Pin_9)
- net GPIO7: now also J3.10 (Pin_10)
- net GPIO8: now also J3.11 (Pin_11)
- net GPIO9: now also J3.12 (Pin_12)
- net RUN: now also J4.10 (Pin_10)
- net VBUS: now also J4.20 (Pin_20)
- net at C18.2, D1.1 (K), R8.1: now also J4.19 (Pin_19)
- net SCL renamed GPIO22
- net GPIO22: now also J4.9 (Pin_9)
- net SDA renamed GPIO21
- net GPIO21: now also J4.7 (Pin_7)
