File: PCB files/Devboard.kicad_pcb (KiCad board)
At the start: 2 copper layers, 42.1 x 52.1 mm, 37 parts, among them J1 USB_C_Receptacle_USB2.0_14P, J2 Conn_01x03, J3 Conn_01x20, J4 Conn_01x20, J5 JST_2mm_LiPo, SW1 SW_Push, U1 RP2040, U2 NCP1117-3.3_SOT223, U3 W25Q128JVS, Y1 12Mhz

Commit message: added MPU-6500 IMU
Parts:
- added C19: 10nF, PCM_SparkFun-Capacitor:C_0603_1608Metric, F.Cu at (209.4, 62.9)
- added C20: 0.1uF, PCM_SparkFun-Capacitor:C_0603_1608Metric, F.Cu at (212.3, 66.8)
- added C21: 0.1uF, PCM_SparkFun-Capacitor:C_0603_1608Metric, F.Cu at (209.6, 69.2)
- added IC1: MPU-6500, KiCadMPU:QFN40P300X300X95-25N-D, F.Cu at (209.4, 66.2)
- moved C13 1.60 mm to (209.8, 72.1), turned to 180 degrees
Routing:
- net /GPIO21: track 16.6 -> 53.2 mm, vias 1 -> 5
- net /GPIO22: track 16.2 -> 47.3 mm, vias 1 -> 5
- net 3.3V: track 8.72 -> 28.9 mm
- net GND: track 67.1 -> 84.5 mm, vias 25 -> 29
- net Net-(IC1-REGOUT): track 0.00 -> 1.41 mm
